File: labs/lab_03/schematics/Transimpedance Ampifier/Lab3TransimpedanceSchematics.kicad_sch (KiCad schematic)
At the start: 3 parts, among them U1 MCP6004

Commit message: Update component values to match lab
Parts:
- Rf: value ??? -> 10M
Changed lines of the file:
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@@
       (effects (font (size 1.27 1.27)))
     )
-    (property "Value" "???" (at 151.13 90.17 90)
+    (property "Value" "10M" (at 151.13 90.17 90)
       (effects (font (size 1.27 1.27)))
     )
