File: labs/lab_04/thermistor/ThermistorSchematic/ThermistorSchematic.kicad_sch (KiCad schematic)
At the start: 12 parts, among them U1 MCP601-xSN, U2 MCP601-xSN

Commit message: Update schematic
Parts:
- removed C1: 100nF, symbol Device:C
- removed C2: 10uF, symbol Device:C_Polarized_US
- removed R3, R4: R_US, symbol Device:R_US
- added C1: 10uF, symbol Device:C_Polarized_US
- added C2: 100nF, symbol Device:C
- added R1: 15k, symbol Device:R_US
- added Rf: 6.8k, symbol Device:R_US
- R2: value R_US -> 5k
- Rd: renamed from R; value R_US -> 27k
- Ri: renamed from R1; value R_US -> 2.2k
- U1, U2: value MCP601-xSN -> MCP601
- renumbered RT to Rt
Connections:
- net +5V: now also C1.1, C2.1, R1.1
- net GND: now also R2.2, C1.2, C2.2
- net Vout: now also Rf.2; no longer R2.2
- net at U1.3 (+): now also R2.1, R1.2
- net at Ri.2, U1.2 (-): now also Rf.1; no longer R2.1
- net at Rd.1, Rt.2: now also Ri.1, U2.2 (-), U2.6; no longer U2.3 (+)
Other:
- moved on the sheet: Rd, Rt

Commit message: schematic
Other:
- note added: "Rt=R0exp(B(1/T-1/T0)) Vin=Rd/(Rd+Rt) Vout=(R2/(R1+R2))(1+Rf/Ri)Vdc-(Rf/Ri)Vin"
Changed lines of the file:
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@@
     (stroke (width 0) (type default))
+  )
+  (text "Rt=R0exp(B(1/T-1/T0))\nVin=Rd/(Rd+Rt)\nVout=(R2/(R1+R2))(1+Rf/Ri)Vdc-(Rf/Ri)Vin"
+    (at 99.06 147.32 0)
+    (effects (font (size 2 2)) (justify left bottom))
   )
   (label "Vout" (at 195.58 104.14 0) (fields_autoplaced)
