File: project/electrical/pressure/PressureSensorSchematic/PressureSensorSchematic.kicad_sch (KiCad schematic)
At the start: 11 parts, among them U1 MCP601, U2 MPXA6115A

Commit message: Pressure sensor clean up
Parts:
- removed R3: 470k, symbol Device:R_US
- removed R4: 122k, symbol Device:R_US
- added R1: 30k, symbol Device:R_US
- added Rf: 33k, symbol Device:R_US
- R2: value 330k -> 10k
- Ri: renamed from R1; value 110k -> 10k
- U2: value MPXA6115A -> MPX5700
Connections:
- net GND is gone; now on net +5V: C1.2, C2.2, C3.1, C4.1, C5.1, U1.4 (V-), U2.3 (GND)
- net +5V: now also R2.1, R1.1; no longer C1.1, C2.1, U1.7 (V+)
- net Vin: now also Ri.1; no longer U1.3 (+)
- net Vout: now also Rf.2; no longer R2.2
- net at Ri.2, U1.2 (-): now also Rf.1; no longer R2.1
- new net: C1.1, C2.1, U1.7 (V+)
- new net: R1.2, R2.2, U1.3 (+)
Other:
- note added: "Vout = (R2/(R1+R2))(1+Rf/Ri) * Vdc - (Rf/Ri) * Vin"
- moved on the sheet: C1, C2, Ri, U1
