File: project/salinity/Salinity_Sensor_Schematic/Salinity_Sensor_Schematic.kicad_sch (KiCad schematic)
At the start: 12 parts, among them U2 MCP6001-OT, U3 MCP6001-OT, U3 U1, U4 MCP6001-OT

Commit message: Updated Values
Parts:
- C1: value C -> 0.004 nF
- R3, R4: value R_US -> 10.4 Ω
- R5: value R_US -> 10.2 Ω
Changed lines of the file:
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@@
       (effects (font (size 1.27 1.27)))
     )
-    (property "Value" "R_US" (at 101.6 72.39 90)
+    (property "Value" "10.4 Ω" (at 101.6 72.39 90)
       (effects (font (size 1.27 1.27)))
     )
@@
   )
   (symbol (lib_id "Device:C") (at 105.41 82.55 0) (unit 1)
-    (in_bom yes) (on_board yes) (dnp no) (fields_autoplaced)
+    (in_bom yes) (on_board yes) (dnp no)
     (property "Reference" "C1" (at 109.22 81.28 0)
       (effects (font (size 1.27 1.27)) (justify left))
     )
-    (property "Value" "C" (at 109.22 83.82 0)
+    (property "Value" "0.004 nF" (at 107.95 78.74 0)
       (effects (font (size 1.27 1.27)) (justify left))
     )
@@
       (effects (font (size 1.27 1.27)))
     )
-    (property "Value" "R_US" (at 180.34 74.93 90)
+    (property "Value" "10.2 Ω" (at 180.34 74.93 90)
       (effects (font (size 1.27 1.27)))
     )
@@
       (effects (font (size 1.27 1.27)))
     )
-    (property "Value" "R_US" (at 140.97 74.93 90)
-      (effects (font (size 1.27 1.27)))
-    )
+    (property "Value" "10.4 Ω" (at 140.97 74.93 90)
+      (effects (font (size 1.27 1.27)))
+    )
