File: project/electrical/salinity/ideal_salinity_schematics/ideal_wavegen_salinity.kicad_sch (KiCad schematic)
At the start: 12 parts, among them U2 MCP6001-OT, U3 MCP6001-OT, U3 U1, U4 MCP6001-OT

Commit message: updated ideal salinity schematics
Parts:
- C1, C2: value 0.004 nF -> 4pF
- C3: value 0.004 nF -> 4 pF
- R1: value R_US -> 2MΩ
- R2: value R_US -> 15kΩ
- R3, R4: value 10.4 Ω -> 10Ω
- R5: value 10.2 Ω -> 10Ω
Changed lines of the file:
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@@
       (effects (font (size 1.27 1.27)))
     )
-    (property "Value" "10.4 Ω" (at 101.6 72.39 90)
+    (property "Value" "10Ω" (at 101.6 72.39 90)
       (effects (font (size 1.27 1.27)))
     )
@@
     (pin "2")
     (instances
-      (project "Salinity_Sensor_Schematic"
+      (project "ideal_wavegen_salinity"
         (path "/9350a783-333a-41b8-a266-5853336ae98e"
           (reference "R3") (unit 1)
@@
       (effects (font (size 1.27 1.27)))
     )
-    (property "Value" "R_US" (at 64.77 50.8 90)
+    (property "Value" "2MΩ" (at 64.77 50.8 90)
       (effects (font (size 1.27 1.27)))
     )
@@
     (pin "2")
     (instances
-      (project "Salinity_Sensor_Schematic"
+      (project "ideal_wavegen_salinity"
         (path "/9350a783-333a-41b8-a266-5853336ae98e"
           (reference "R1") (unit 1)
@@
       (effects (font (size 1.27 1.27)) (justify left))
     )
-    (property "Value" "0.004 nF" (at 187.96 83.82 0)
+    (property "Value" "4 pF" (at 187.96 83.82 0)
       (effects (font (size 1.27 1.27)) (justify left))
     )
@@
     (pin "2")
     (instances
-      (project "Salinity_Sensor_Schematic"
+      (project "ideal_wavegen_salinity"
         (path "/9350a783-333a-41b8-a266-5853336ae98e"
           (reference "C3") (unit 1)
@@
     (pin "1")
     (instances
-      (project "Salinity_Sensor_Schematic"
+      (project "ideal_wavegen_salinity"
         (path "/9350a783-333a-41b8-a266-5853336ae98e"
           (reference "#PWR08") (unit 1)
@@
       (effects (font (size 1.27 1.27)) (justify left))
     )
-    (property "Value" "0.004 nF" (at 148.59 86.36 0)
+    (property "Value" "4pF" (at 148.59 86.36 0)
       (effects (font (size 1.27 1.27)) (justify left))
     )
@@
     (pin "1")
     (instances
-      (project "Salinity_Sensor_Schematic"
+      (project "ideal_wavegen_salinity"
         (path "/9350a783-333a-41b8-a266-5853336ae98e"
           (reference "C2") (unit 1)
@@
     (pin "1")
     (instances
-      (project "Salinity_Sensor_Schematic"
+      (project "ideal_wavegen_salinity"
         (path "/9350a783-333a-41b8-a266-5853336ae98e"
           (reference "#PWR01") (unit 1)
@@
     (pin "2")
     (instances
-      (project "Salinity_Sensor_Schematic"
+      (project "ideal_wavegen_salinity"
         (path "/9350a783-333a-41b8-a266-5853336ae98e"
           (reference "U4") (unit 1)
@@
       (effects (font (size 1.27 1.27)) (justify left))
     )
-    (property "Value" "0.004 nF" (at 107.95 78.74 0)
+    (property "Value" "4pF" (at 107.95 83.82 0)
       (effects (font (size 1.27 1.27)) (justify left))
     )
@@
     (pin "1")
     (instances
-      (project "Salinity_Sensor_Schematic"
+      (project "ideal_wavegen_salinity"
         (path "/9350a783-333a-41b8-a266-5853336ae98e"
           (reference "C1") (unit 1)
@@
     (pin "1")
     (instances
-      (project "Salinity_Sensor_Schematic"
+      (project "ideal_wavegen_salinity"
         (path "/9350a783-333a-41b8-a266-5853336ae98e"
           (reference "#PWR09") (unit 1)
@@
       (effects (font (size 1.27 1.27)))
     )
-    (property "Value" "10.2 Ω" (at 180.34 74.93 90)
+    (property "Value" "10Ω" (at 180.34 74.93 90)
       (effects (font (size 1.27 1.27)))
     )
@@
     (pin "1")
     (instances
-      (project "Salinity_Sensor_Schematic"
+      (project "ideal_wavegen_salinity"
         (path "/9350a783-333a-41b8-a266-5853336ae98e"
           (reference "R5") (unit 1)
@@
     (pin "1")
     (instances
-      (project "Salinity_Sensor_Schematic"
+      (project "ideal_wavegen_salinity"
         (path "/9350a783-333a-41b8-a266-5853336ae98e"
           (reference "#PWR011") (unit 1)
@@
     (pin "5")
     (instances
-      (project "Salinity_Sensor_Schematic"
+      (project "ideal_wavegen_salinity"
         (path "/9350a783-333a-41b8-a266-5853336ae98e"
           (reference "U3") (unit 1)
@@
       (effects (font (size 1.27 1.27)))
     )
-    (property "Value" "R_US" (at 48.26 67.31 90)
+    (property "Value" "15kΩ" (at 48.26 67.31 90)
       (effects (font (size 1.27 1.27)))
     )
@@
     (pin "1")
     (instances
-      (project "Salinity_Sensor_Schematic"
+      (project "ideal_wavegen_salinity"
         (path "/9350a783-333a-41b8-a266-5853336ae98e"
           (reference "R2") (unit 1)
@@
     (pin "1")
     (instances
-      (project "Salinity_Sensor_Schematic"
+      (project "ideal_wavegen_salinity"
         (path "/9350a783-333a-41b8-a266-5853336ae98e"
           (reference "#PWR02") (unit 1)
@@
       (effects (font (size 1.27 1.27)))
     )
-    (property "Value" "10.4 Ω" (at 140.97 74.93 90)
+    (property "Value" "10Ω" (at 140.97 74.93 90)
       (effects (font (size 1.27 1.27)))
     )
@@
     (pin "2")
     (instances
-      (project "Salinity_Sensor_Schematic"
+      (project "ideal_wavegen_salinity"
         (path "/9350a783-333a-41b8-a266-5853336ae98e"
           (reference "R4") (unit 1)
@@
     (pin "1")
     (instances
-      (project "Salinity_Sensor_Schematic"
+      (project "ideal_wavegen_salinity"
         (path "/9350a783-333a-41b8-a266-5853336ae98e"
           (reference "#PWR010") (unit 1)
@@
     (pin "1")
     (instances
-      (project "Salinity_Sensor_Schematic"
+      (project "ideal_wavegen_salinity"
         (path "/9350a783-333a-41b8-a266-5853336ae98e"
           (reference "#PWR07") (unit 1)
@@
     (pin "1")
     (instances
-      (project "Salinity_Sensor_Schematic"
+      (project "ideal_wavegen_salinity"
         (path "/9350a783-333a-41b8-a266-5853336ae98e"
           (reference "#PWR04") (unit 1)
@@
     (pin "1")
     (instances
-      (project "Salinity_Sensor_Schematic"
+      (project "ideal_wavegen_salinity"
         (path "/9350a783-333a-41b8-a266-5853336ae98e"
           (reference "#PWR05") (unit 1)
@@
     (pin "1")
     (instances
-      (project "Salinity_Sensor_Schematic"
+      (project "ideal_wavegen_salinity"
         (path "/9350a783-333a-41b8-a266-5853336ae98e"
           (reference "#PWR06") (unit 1)
@@
     (pin "5")
     (instances
-      (project "Salinity_Sensor_Schematic"
+      (project "ideal_wavegen_salinity"
         (path "/9350a783-333a-41b8-a266-5853336ae98e"
           (reference "U3") (unit 1)
@@
     (pin "1")
     (instances
-      (project "Salinity_Sensor_Schematic"
+      (project "ideal_wavegen_salinity"
         (path "/9350a783-333a-41b8-a266-5853336ae98e"
           (reference "#PWR012") (unit 1)
@@
     (pin "1")
     (instances
-      (project "Salinity_Sensor_Schematic"
+      (project "ideal_wavegen_salinity"
         (path "/9350a783-333a-41b8-a266-5853336ae98e"
           (reference "#PWR03") (unit 1)
@@
     (pin "4")
     (instances
-      (project "Salinity_Sensor_Schematic"
+      (project "ideal_wavegen_salinity"
         (path "/9350a783-333a-41b8-a266-5853336ae98e"
           (reference "U2") (unit 1)

Commit message: Made some circuits better for overleaf
Other:
- moved on the sheet: C1, C2, C3, R1, R2, R3, R4, R5, U2, U3, U4
