File: project/electrical/temperature/thermistor/ThermistorSchematic/ThermistorSchematic.kicad_sch (KiCad schematic)
At the start: 12 parts, among them U1 MCP601, U2 MCP601

Commit message: updated temperature circuit, moved salinity circuit
Parts:
- R2: value 30k -> 10k
Connections:
- net at U2.3 (+): now also Rd.1, Rt.2
- net Vin: 2.7  to 3.3 V renamed Vin: 1.2 to 1.7 V
- net Vin: 1.2 to 1.7 V: no longer Rd.1, Rt.2
- net Vout: 0.2 to 3.0 V renamed Vout: 0.4 to 2.8 V
Other:
- moved on the sheet: Rd, Rt
Changed lines of the file:
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@@
   (junction (at 166.37 111.76) (diameter 0) (color 0 0 0 0)
   )
-  (junction (at 86.36 91.44) (diameter 0) (color 0 0 0 0)
+  (junction (at 86.36 96.52) (diameter 0) (color 0 0 0 0)
   )
   (junction (at 101.6 116.84) (diameter 0) (color 0 0 0 0)
@@
   (junction (at 156.21 93.98) (diameter 0) (color 0 0 0 0)
   )
-  (junction (at 93.98 91.44) (diameter 0) (color 0 0 0 0)
-  )
   (junction (at 101.6 110.49) (diameter 0) (color 0 0 0 0)
   )
@@
     (stroke (width 0) (type default))
   )
+  (wire (pts (xy 86.36 96.52) (xy 96.52 96.52))
+    (stroke (width 0) (type default))
+  )
   (wire (pts (xy 172.72 78.74) (xy 180.34 78.74))
     (stroke (width 0) (type default))
@@
   )
   (wire (pts (xy 154.94 111.76) (xy 139.7 111.76))
-    (stroke (width 0) (type default))
-  )
-  (wire (pts (xy 86.36 91.44) (xy 93.98 91.44))
     (stroke (width 0) (type default))
   )
@@
     (effects (font (size 2 2)) (justify left bottom))
   )
-  (label "Vin: 2.7  to 3.3 V" (at 116.84 93.98 0) (fields_autoplaced)
+  (label "Vin: 1.2 to 1.7 V" (at 116.84 93.98 0) (fields_autoplaced)
     (effects (font (size 1.27 1.27)) (justify left bottom))
   )
-  (label "Vout: 0.2 to 3.0 V" (at 198.12 104.14 0) (fields_autoplaced)
+  (label "Vout: 0.4 to 2.8 V" (at 198.12 104.14 0) (fields_autoplaced)
     (effects (font (size 1.27 1.27)) (justify left bottom))
   )
@@
     )
   )
-  (symbol (lib_id "power:GND") (at 86.36 99.06 0) (mirror y) (unit 1)
-    (in_bom yes) (on_board yes) (dnp no) (fields_autoplaced)
-    (property "Reference" "#PWR07" (at 86.36 105.41 0)
-      (effects (font (size 1.27 1.27)) hide)
-    )
-    (property "Value" "GND" (at 86.36 104.14 0)
-      (effects (font (size 1.27 1.27)))
-    )
-    (property "Footprint" "" (at 86.36 99.06 0)
-      (effects (font (size 1.27 1.27)) hide)
-    )
-    (property "Datasheet" "" (at 86.36 99.06 0)
+  (symbol (lib_id "power:GND") (at 86.36 104.14 0) (mirror y) (unit 1)
+    (in_bom yes) (on_board yes) (dnp no) (fields_autoplaced)
+    (property "Reference" "#PWR07" (at 86.36 110.49 0)
+      (effects (font (size 1.27 1.27)) hide)
+    )
+    (property "Value" "GND" (at 86.36 109.22 0)
+      (effects (font (size 1.27 1.27)))
+    )
+    (property "Footprint" "" (at 86.36 104.14 0)
+      (effects (font (size 1.27 1.27)) hide)
+    )
+    (property "Datasheet" "" (at 86.36 104.14 0)
       (effects (font (size 1.27 1.27)) hide)
     )
@@
     )
   )
-  (symbol (lib_id "power:+5V") (at 86.36 83.82 0) (mirror y) (unit 1)
-    (in_bom yes) (on_board yes) (dnp no) (fields_autoplaced)
-    (property "Reference" "#PWR06" (at 86.36 87.63 0)
-      (effects (font (size 1.27 1.27)) hide)
-    )
-    (property "Value" "+5V" (at 86.36 78.74 0)
-      (effects (font (size 1.27 1.27)))
-    )
-    (property "Footprint" "" (at 86.36 83.82 0)
-      (effects (font (size 1.27 1.27)) hide)
-    )
-    (property "Datasheet" "" (at 86.36 83.82 0)
+  (symbol (lib_id "power:+5V") (at 86.36 88.9 0) (mirror y) (unit 1)
+    (in_bom yes) (on_board yes) (dnp no) (fields_autoplaced)
+    (property "Reference" "#PWR06" (at 86.36 92.71 0)
+      (effects (font (size 1.27 1.27)) hide)
+    )
+    (property "Value" "+5V" (at 86.36 83.82 0)
+      (effects (font (size 1.27 1.27)))
+    )
+    (property "Footprint" "" (at 86.36 88.9 0)
+      (effects (font (size 1.27 1.27)) hide)
+    )
+    (property "Datasheet" "" (at 86.36 88.9 0)
       (effects (font (size 1.27 1.27)) hide)
     )
@@
       (effects (font (size 1.27 1.27)) (justify left))
     )
-    (property "Value" "30k" (at 133.35 119.38 0)
+    (property "Value" "10k" (at 133.35 119.38 0)
       (effects (font (size 1.27 1.27)) (justify left))
     )
@@
     )
   )
-  (symbol (lib_id "Device:R_US") (at 86.36 87.63 0) (mirror y) (unit 1)
-    (in_bom yes) (on_board yes) (dnp no) (fields_autoplaced)
-    (property "Reference" "Rt" (at 83.82 86.36 0)
-      (effects (font (size 1.27 1.27)) (justify left))
-    )
-    (property "Value" "R_US" (at 83.82 88.9 0)
+  (symbol (lib_id "Device:R_US") (at 86.36 92.71 0) (mirror y) (unit 1)
+    (in_bom yes) (on_board yes) (dnp no) (fields_autoplaced)
+    (property "Reference" "Rt" (at 83.82 91.44 0)
+      (effects (font (size 1.27 1.27)) (justify left))
+    )
+    (property "Value" "R_US" (at 83.82 93.98 0)
       (effects (font (size 1.27 1.27)) (justify left) hide)
     )
-    (property "Footprint" "" (at 85.344 87.884 90)
-      (effects (font (size 1.27 1.27)) hide)
-    )
-    (property "Datasheet" "~" (at 86.36 87.63 0)
+    (property "Footprint" "" (at 85.344 92.964 90)
+      (effects (font (size 1.27 1.27)) hide)
+    )
+    (property "Datasheet" "~" (at 86.36 92.71 0)
       (effects (font (size 1.27 1.27)) hide)
     )
@@
     )
   )
-  (symbol (lib_id "Device:R_US") (at 86.36 95.25 0) (mirror y) (unit 1)
-    (in_bom yes) (on_board yes) (dnp no) (fields_autoplaced)
-    (property "Reference" "Rd" (at 83.82 93.98 0)
-      (effects (font (size 1.27 1.27)) (justify left))
-    )
-    (property "Value" "27k" (at 83.82 96.52 0)
-      (effects (font (size 1.27 1.27)) (justify left))
-    )
-    (property "Footprint" "" (at 85.344 95.504 90)
-      (effects (font (size 1.27 1.27)) hide)
-    )
-    (property "Datasheet" "~" (at 86.36 95.25 0)
-      (effects (font (size 1.27 1.27)) hide)
-    )
+  (symbol (lib_id "Device:R_US") (at 86.36 100.33 0) (mirror y) (unit 1)
+    (in_bom yes) (on_board yes) (dnp no) (fields_autoplaced)
+    (property "Reference" "Rd" (at 83.82 99.06 0)
+      (effects (font (size 1.27 1.27)) (justify left))
+    )
+    (property "Value" "27k" (at 83.82 101.6 0)
+      (effects (font (size 1.27 1.27)) (justify left))
+    )
+    (property "Footprint" "" (at 85.344 100.584 90)
+      (effects (font (size 1.27 1.27)) hide)
+    )
+    (property "Datasheet" "~" (at 86.36 100.33 0)
+      (effects (font (size 1.27 1.27)) hide)
+    )

Commit message: Made some circuits better for overleaf
Connections:
- net Vin: 1.2 to 1.7 V: no longer names the net of Ri.1, U2.2 (-), U2.6
- net Vout: 0.4 to 2.8 V: no longer names the net of Rf.2, U1.6
Other:
- note added: "Vin: 1.2 to 1.7 V"
- note added: "Vout: 0.4 to 2.8 V"
- moved on the sheet: C1, C2, C3, C4, R1, R2, Rd, Rf, Ri, Rt, U2
